Commit message: gazebo world with control plugin

File: src/yuen_bot/urdf/fishbot/actuator/caster.urdf.xacro (robot description, xacro)
@@ -24,4 +24,10 @@
             <xacro:sphere_inertia m="0.05" r="0.016"/>
         </link>
+        <gazebo reference="${caster_name}_caster_link">
+            <mu1 value="0.0" />
+            <mu2 value="0.0" />
+            <kp value="1000000000.0" />
+            <kd value="1.0" />
+        </gazebo>
         <joint name="${caster_name}_caster_joint" type="fixed">
             <parent link="base_link" />

File: src/yuen_bot/urdf/fishbot/actuator/wheel.urdf.xacro (robot description, xacro)
@@ -24,4 +24,10 @@
 			<xacro:cylinder_inertia m="0.05" r="0.032" h="0.04"/>
 	    </link>
+		<gazebo reference="${wheel_name}_wheel_link">
+			<mu1 value="20.0" />
+			<mu2 value="20.0" />
+			<kp value="1000000000.0" />
+			<kd value="1.0" />
+		</gazebo>
 	    <joint name="${wheel_name}_wheel_joint" type="continuous">
 	    	<parent link="base_link" />

File: src/yuen_bot/urdf/fishbot/fishbot.urdf.xacro (robot description, xacro)
@@ -18,3 +18,6 @@
 	<xacro:laser_xacro xyz="0 0 0.10" />
 	<xacro:camera_xacro xyz="0.10 0 0.075" />
+    <!-- Gazebo 插件 -->
+    <xacro:include filename="$(find yuen_bot)/urdf/fishbot/plugins/gazebo_control_plugin.xacro"/>
+    <xacro:gazebo_control_plugin/>
 </robot>

File: src/yuen_bot/urdf/fishbot/sensor/laser.urdf.xacro (robot description, xacro)
@@ -3,4 +3,10 @@
 	<xacro:include filename="$(find yuen_bot)/urdf/fishbot/inertia.urdf.xacro"/>
 	<xacro:macro name="laser_xacro" params="xyz">
+	<gazebo reference="laser_cylinder_link">
+		<material>Gazebo/Black</material>
+	</gazebo>
+	<gazebo reference="laser_link">
+		<material>Gazebo/Black</material>
+	</gazebo>
 	<!-- ============雷达支撑杆 ================ -->
 		<link name="laser_cylinder_link">
