Commit message: all the xacros and launch settings in chapter6

File: src/yuen_bot/urdf/fishbot/fishbot.urdf.xacro (robot description, xacro)
@@ -23,3 +23,6 @@
     <xacro:include filename="$(find fishbot_description)/urdf/fishbot/plugins/gazebo_sensor_plugin.xacro" />
     <xacro:gazebo_sensor_plugin />
+    <!-- <xacro:gazebo_control_plugin /> -->
+    <xacro:include filename="$(find fishbot_description)/urdf/fishbot/fishbot.ros2_control.xacro" />
+    <xacro:fishbot_ros2_control />
 </robot>

File: src/yuen_bot/urdf/fishbot/plugins/gazebo_sensor_plugin.xacro (robot description, xacro)
@@ -42,4 +42,97 @@
         </sensor>
     </gazebo>
+    <gazebo reference="imu_link">
+        <sensor name="imu_sensor" type="imu">
+            <plugin name="imu_plugin" filename="libgazebo_ros_imu_sensor.so">
+                <ros>
+                    <namespace>/</namespace>
+                <remapping>~/out:=imu</remapping>
+                </ros>
+                <initial_orientation_as_reference>false</initial_orientation_as_reference>
+            </plugin>
+            <update_rate>100</update_rate>
+            <always_on>true</always_on>
+            <!-- 六轴噪声设置 -->
+            <imu>
+                <angular_velocity>
+                    <x>
+                        <noise type="gaussian">
+                            <mean>0.0</mean>
+                            <stddev>2e-4</stddev>
+                            <bias_mean>0.0000075</bias_mean>
+                            <bias_stddev>0.0000008</bias_stddev>
+                        </noise>
+                    </x>
+                    <y>
+                        <noise type="gaussian">
+                            <mean>0.0</mean>
+                            <stddev>2e-4</stddev>
+                            <bias_mean>0.0000075</bias_mean>
+                            <bias_stddev>0.0000008</bias_stddev>
+                        </noise>
+                    </y>
+                    <z>
+                        <noise type="gaussian">
+                            <mean>0.0</mean>
+                            <stddev>2e-4</stddev>
+                            <bias_mean>0.0000075</bias_mean>
+                            <bias_stddev>0.0000008</bias_stddev>
+                        </noise>
+                    </z>
+                </angular_velocity>
+                <linear_acceleration>
+                    <x>
+                        <noise type="gaussian">
+                            <mean>0.0</mean>
+                            <stddev>1.7e-2</stddev>
+                            <bias_mean>0.1</bias_mean>
+                            <bias_stddev>0.001</bias_stddev>
+                        </noise>
+                    </x>
+                    <y>
+                        <noise type="gaussian">
+                            <mean>0.0</mean>
+                            <stddev>1.7e-2</stddev>
+                            <bias_mean>0.1</bias_mean>
+                            <bias_stddev>0.001</bias_stddev>
+                        </noise>
+                    </y>
+                    <z>
+                        <noise type="gaussian">
+                            <mean>0.0</mean>
+                            <stddev>1.7e-2</stddev>
+                            <bias_mean>0.1</bias_mean>
+                            <bias_stddev>0.001</bias_stddev>
+                        </noise>
+                    </z>
+                </linear_acceleration>
+            </imu>
+        </sensor>
+    </gazebo>
+    <gazebo reference="camera_link">
+        <sensor type="depth" name="camera_sensor">
+          <plugin name="depth_camera" filename="libgazebo_ros_camera.so">
+                <frame_name>camera_optical_link</frame_name>
+          </plugin>
+          <always_on>true</always_on>
+          <update_rate>10</update_rate>
+            <camera name="camera">
+                <horizontal_fov>1.5009831567</horizontal_fov>
+                <image>
+                    <width>800</width>
+                    <height>600</height>
+                    <format>R8G8B8</format>
+                </image>
+                <distortion>
+                    <k1>0.0</k1>
+                    <k2>0.0</k2>
+                    <k3>0.0</k3>
+                    <p1>0.0</p1>
+                    <p2>0.0</p2>
+                    <center>0.5 0.5</center>
+                </distortion>
+            </camera>
+        </sensor>
+    </gazebo>
 </xacro:macro>
 </robot>

File: src/yuen_bot/urdf/fishbot/sensor/camera.urdf.xacro (robot description, xacro)
@@ -25,4 +25,10 @@
 			<xacro:box_inertia m="0.1" w="0.02" h="0.10" d="0.02"/>
 		</link>
+		<link name="camera_optical_link"></link>
+		<joint name="camera_optical_joint" type="fixed">
+			<parent link="camera_link" />
+			<child link="camera_optical_link" />
+			<origin xyz="0 0 0" rpy="${-pi/2} 0 ${-pi/2}" />
+		</joint>
 		<joint name="camera_joint" type="fixed">
 			<parent link="base_link" />
